File: OefenPrintplaat/OefenPrintplaat.kicad_pcb (KiCad board)
At the start: 2 copper layers, 20 x 20 mm, 3 parts

Commit message: update oefenprintplaat
Routing:
- net GND: track 0.00 -> 7.72 mm, vias 0 -> 1
- net VCC: track 0.00 -> 5.24 mm
- net Net-(D1-A): track 0.00 -> 2.35 mm
- added copper zone on B.Cu, net GND
- added copper zone on F.Cu, net VCC
Other:
- board size 20 x 20 mm -> 12 x 11.5 mm
Changed lines of the file:
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@@
 		(tags "LED")
 		(property "Reference" "D1"
-			(at 0 -1.43 360)
+			(at 0 -1.43 0)
 			(layer "F.SilkS")
 			(effects
@@
 		)
 		(property "Value" "RED"
-			(at 0 1.43 360)
+			(at 0 1.43 0)
 			(layer "F.Fab")
 			(effects
@@
 		)
 		(fp_text user "${REFERENCE}"
-			(at 0 0 360)
+			(at 0 0 0)
 			(layer "F.Fab")
 			(effects
@@
 	(gr_rect
 		(start 76 33)
-		(end 96 53)
+		(end 88 44.5)
 		(stroke
 			(width 0.05)
@@
 		(layer "Edge.Cuts")
 	)
+	(segment
+		(start 84.575 39.575)
+		(end 84.5 39.5)
+		(width 0.2)
+		(layer "F.Cu")
+		(net 1)
+	)
+	(segment
+		(start 84.575 42)
+		(end 84.575 39.575)
+		(width 0.2)
+		(layer "F.Cu")
+		(net 1)
+	)
+	(via
+		(at 84.5 39.5)
+		(size 0.6)
+		(drill 0.3)
+		(layers "F.Cu" "B.Cu")
+		(free yes)
+		(net 1)
+	)
+	(segment
+		(start 84.5 39.5)
+		(end 83.625 38.625)
+		(width 0.2)
+		(layer "B.Cu")
+		(net 1)
+	)
+	(segment
+		(start 83.625 38.625)
+		(end 83.625 34.675)
+		(width 0.2)
+		(layer "B.Cu")
+		(net 1)
+	)
+	(segment
+		(start 79 38.7)
+		(end 80.375 37.325)
+		(width 0.2)
+		(layer "F.Cu")
+		(net 2)
+	)
+	(segment
+		(start 79 42)
+		(end 79 38.7)
+		(width 0.2)
+		(layer "F.Cu")
+		(net 2)
+	)
+	(segment
+		(start 80.65 42)
+		(end 83 42)
+		(width 0.2)
+		(layer "F.Cu")
+		(net 3)
+	)
+	(zone
+		(net 2)
+		(net_name "VCC")
+		(layer "F.Cu")
+		(hatch edge 0.5)
+		(connect_pads
+			(clearance 0.5)
+		)
+		(min_thickness 0.25)
+		(filled_areas_thickness no)
+		(fill yes
+			(thermal_gap 0.5)
+			(thermal_bridge_width 0.5)
+		)
+		(polygon
+			(pts
+				(xy 76 33) (xy 88 33) (xy 88 44.5) (xy 76 44.5)
+			)
+		)
+	)
+	(zone
+		(net 1)
+		(net_name "GND")
+		(layer "B.Cu")
+		(hatch edge 0.5)
+		(priority 2)
+		(connect_pads
+			(clearance 0.5)
+		)
+		(min_thickness 0.25)
+		(filled_areas_thickness no)
+		(fill yes
+			(thermal_gap 0.5)
+			(thermal_bridge_width 0.5)
+		)
+		(polygon
+			(pts
+				(xy 76 33) (xy 88 33) (xy 88 44.5) (xy 76 44.5)
+			)
+		)
+	)
 )
