File: Puzzle1/puzzle1/GPIO1.kicad_sch (KiCad schematic)
At the start: 2 parts, among them U1 PCA9555D

Commit message: update after review
Changed lines of the file:
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@@
 		)
 	)
-	(label "GPIO_[1..16]"
+	(label "GPIO_[1..96]"
 		(at 137.16 81.28 0)
 		(fields_autoplaced yes)
@@
 		)
 	)
-	(hierarchical_label "GPIO_[1..16]"
+	(hierarchical_label "GPIO_[1..96]"
 		(shape bidirectional)
 		(at 152.4 81.28 0)
