File: Puzzle1/puzzle1/GPIOExpanderMain.kicad_sch (KiCad schematic)
At the start: 0 parts

Commit message: update after review
Other:
- sheet GPIOx40 ports: added GPIO_[1..96]; removed GPIO_[1..16]
- sheet GPIOx42 ports: added GPIO_[1..96]; removed GPIO_[17..32]
- sheet GPIOx44 ports: added GPIO_[1..96]; removed GPIO_[33..48]
- sheet GPIOx46 ports: added GPIO_[1..96]; removed GPIO_[49..64]
- sheet GPIOx48 ports: added GPIO_[1..96]; removed GPIO_[65..80]
- sheet GPIOx4A ports: added GPIO_[1..96]; removed GPIO_[81..96]
Changed lines of the file:
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@@
 	(bus
 		(pts
-			(xy 190.5 52.07) (xy 204.47 52.07)
-		)
-		(stroke
-			(width 0)
-			(type default)
-		)
-	)
-	(wire
-		(pts
-			(xy 200.66 38.1) (xy 204.47 38.1)
+			(xy 130.81 48.26) (xy 144.78 48.26)
+		)
+		(stroke
+			(width 0)
+			(type default)
+		)
+	)
+	(wire
+		(pts
+			(xy 140.97 34.29) (xy 144.78 34.29)
 		)
 		(stroke
@@
 	(wire
 		(pts
-			(xy 200.66 41.91) (xy 204.47 41.91)
+			(xy 140.97 38.1) (xy 144.78 38.1)
 		)
 		(stroke
@@
 	(wire
 		(pts
-			(xy 50.8 111.76) (xy 55.88 111.76)
+			(xy 204.47 34.29) (xy 209.55 34.29)
 		)
 		(stroke
@@
 	(bus
 		(pts
-			(xy 41.91 124.46) (xy 55.88 124.46)
-		)
-		(stroke
-			(width 0)
-			(type default)
-		)
-	)
-	(wire
-		(pts
-			(xy 50.8 115.57) (xy 55.88 115.57)
+			(xy 195.58 46.99) (xy 209.55 46.99)
+		)
+		(stroke
+			(width 0)
+			(type default)
+		)
+	)
+	(wire
+		(pts
+			(xy 204.47 38.1) (xy 209.55 38.1)
 		)
 		(stroke
@@
 	)
 	(label "SDA"
-		(at 50.8 111.76 0)
+		(at 204.47 34.29 0)
 		(fields_autoplaced yes)
 		(effects
@@
 	)
 	(label "GPIO_[1..96]"
-		(at 43.18 124.46 0)
+		(at 196.85 46.99 0)
 		(fields_autoplaced yes)
 		(effects
@@
 	)
 	(label "SCL"
-		(at 200.66 41.91 0)
+		(at 140.97 38.1 0)
 		(fields_autoplaced yes)
 		(effects
@@
 	)
 	(label "SDA"
-		(at 200.66 38.1 0)
+		(at 140.97 34.29 0)
 		(fields_autoplaced yes)
 		(effects
@@
 	)
 	(label "GPIO_[1..96]"
-		(at 191.77 52.07 0)
+		(at 132.08 48.26 0)
 		(fields_autoplaced yes)
 		(effects
@@
 	)
 	(label "SCL"
-		(at 50.8 115.57 0)
+		(at 204.47 38.1 0)
 		(fields_autoplaced yes)
 		(effects
@@
 			)
 		)
-		(pin "GPIO_[17..32]" bidirectional
+		(pin "GPIO_[1..96]" bidirectional
 			(at 90.17 46.99 180)
 			(effects
@@
 	)
 	(sheet
-		(at 204.47 24.13)
+		(at 144.78 20.32)
 		(size 34.29 43.18)
 		(fields_autoplaced yes)
@@
 		)
 		(property "Sheetname" "GPIOx44"
-			(at 204.47 23.4184 0)
+			(at 144.78 19.6084 0)
 			(effects
 				(font
@@
 		)
 		(property "Sheetfile" "GPIO3.kicad_sch"
-			(at 204.47 67.8946 0)
+			(at 144.78 64.0846 0)
 			(effects
 				(font
@@
 		)
 		(pin "SDA" bidirectional
-			(at 204.47 38.1 180)
+			(at 144.78 34.29 180)
 			(effects
 				(font
@@
 		)
 		(pin "SCL" input
-			(at 204.47 41.91 180)
-			(effects
-				(font
-					(size 1.27 1.27)
-				)
-				(justify left)
-			)
-		)
-		(pin "GPIO_[33..48]" bidirectional
-			(at 204.47 52.07 180)
+			(at 144.78 38.1 180)
+			(effects
+				(font
+					(size 1.27 1.27)
+				)
+				(justify left)
+			)
+		)
+		(pin "GPIO_[1..96]" bidirectional
+			(at 144.78 48.26 180)
 			(effects
 				(font
@@
 	)
 	(sheet
-		(at 55.88 97.79)
+		(at 209.55 20.32)
 		(size 34.29 43.18)
 		(fields_autoplaced yes)
@@
 		)
 		(property "Sheetname" "GPIOx46"
-			(at 55.88 97.0784 0)
+			(at 209.55 19.6084 0)
 			(effects
 				(font
@@
 		)
 		(property "Sheetfile" "GPIO4.kicad_sch"
-			(at 55.88 141.5546 0)
+			(at 209.55 64.0846 0)
 			(effects
 				(font
@@
 		)
 		(pin "SDA" bidirectional
-			(at 55.88 111.76 180)
+			(at 209.55 34.29 180)
 			(effects
 				(font
@@
 		)
 		(pin "SCL" input
-			(at 55.88 115.57 180)
-			(effects
-				(font
-					(size 1.27 1.27)
-				)
-				(justify left)
-			)
-		)
-		(pin "GPIO_[49..64]" bidirectional
-			(at 55.88 124.46 180)
+			(at 209.55 38.1 180)
+			(effects
+				(font
+					(size 1.27 1.27)
+				)
+				(justify left)
+			)
+		)
+		(pin "GPIO_[1..96]" bidirectional
+			(at 209.55 46.99 180)
 			(effects
 				(font
@@
 			)
 		)
-		(pin "GPIO_[81..96]" bidirectional
+		(pin "GPIO_[1..96]" bidirectional
 			(at 185.42 120.65 180)
 			(effects
@@
 			)
 		)
-		(pin "GPIO_[65..80]" bidirectional
+		(pin "GPIO_[1..96]" bidirectional
 			(at 115.57 120.65 180)
 			(effects
@@
 			)
 		)
-		(pin "GPIO_[1..16]" bidirectional
+		(pin "GPIO_[1..96]" bidirectional
 			(at 34.29 48.26 180)
 			(effects
