File: Puzzle1/puzzle1/Connectors.kicad_sch (KiCad schematic)
At the start: 19 parts, among them J10 Conn_01x09_Pin, J11 Conn_01x04_Pin, J12 Conn_01x04_Pin, J13 Conn_01x04_Pin, J14 Conn_01x04_Pin, J2 Conn_01x09_Pin, J3 Conn_01x09_Pin, J4 Conn_01x09_Pin, J5 Conn_01x09_Pin, J6 Conn_01x09_Pin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

Commit message: update after review
Parts:
- R3, R4, R5, R6, R7, R8: footprint (none) -> Resistor_SMD:R_0603_1608Metric_Pad0.98x0.95mm_HandSolder
Connections:
- no-connect marks 0 -> 6
Changed lines of the file:
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@@
 		(color 0 0 0 0)
 	)
+	(no_connect
+		(at 97.79 153.67)
+	)
+	(no_connect
+		(at 82.55 153.67)
+	)
+	(no_connect
+		(at 97.79 151.13)
+	)
+	(no_connect
+		(at 82.55 151.13)
+	)
+	(no_connect
+		(at 97.79 148.59)
+	)
+	(no_connect
+		(at 82.55 148.59)
+	)
 	(bus_entry
 		(at 105.41 35.56)
@@
 	)
 	(bus_entry
+		(at 92.71 151.13)
+		(size 2.54 2.54)
+		(stroke
+			(width 0)
+			(type default)
+		)
+	)
+	(bus_entry
 		(at 49.53 63.5)
 		(size -2.54 2.54)
@@
 	)
 	(bus_entry
+		(at 92.71 148.59)
+		(size 2.54 2.54)
+		(stroke
+			(width 0)
+			(type default)
+		)
+	)
+	(bus_entry
 		(at 105.41 93.98)
 		(size -2.54 2.54)
@@
 	)
 	(bus_entry
+		(at 92.71 151.13)
+		(size -2.54 2.54)
+		(stroke
+			(width 0)
+			(type default)
+		)
+	)
+	(bus_entry
 		(at 105.41 63.5)
 		(size -2.54 2.54)
@@
 	)
 	(bus_entry
+		(at 92.71 146.05)
+		(size 2.54 2.54)
+		(stroke
+			(width 0)
+			(type default)
+		)
+	)
+	(bus_entry
 		(at 237.49 33.02)
 		(size -2.54 2.54)
@@
 	)
 	(bus_entry
+		(at 92.71 146.05)
+		(size -2.54 2.54)
+		(stroke
+			(width 0)
+			(type default)
+		)
+	)
+	(bus_entry
 		(at 237.49 38.1)
 		(size -2.54 2.54)
@@
 	)
 	(bus_entry
+		(at 92.71 148.59)
+		(size -2.54 2.54)
+		(stroke
+			(width 0)
+			(type default)
+		)
+	)
+	(bus_entry
 		(at 49.53 88.9)
 		(size -2.54 2.54)
@@
 	(wire
 		(pts
+			(xy 95.25 153.67) (xy 97.79 153.67)
+		)
+		(stroke
+			(width 0)
+			(type default)
+		)
+	)
+	(wire
+		(pts
 			(xy 91.44 30.48) (xy 102.87 30.48)
 		)
@@
 		)
 	)
+	(wire
+		(pts
+			(xy 82.55 148.59) (xy 90.17 148.59)
+		)
+		(stroke
+			(width 0)
+			(type default)
+		)
+	)
 	(bus
 		(pts
@@
 		)
 	)
+	(wire
+		(pts
+			(xy 82.55 151.13) (xy 90.17 151.13)
+		)
+		(stroke
+			(width 0)
+			(type default)
+		)
+	)
 	(bus
 		(pts
@@
 		)
 	)
+	(wire
+		(pts
+			(xy 95.25 148.59) (xy 97.79 148.59)
+		)
+		(stroke
+			(width 0)
+			(type default)
+		)
+	)
 	(bus
 		(pts
@@
 	(bus
 		(pts
+			(xy 92.71 151.13) (xy 92.71 156.21)
+		)
+		(stroke
+			(width 0)
+			(type default)
+		)
+	)
+	(bus
+		(pts
 			(xy 162.56 73.66) (xy 162.56 76.2)
 		)
@@
 		)
 	)
+	(bus
+		(pts
+			(xy 92.71 146.05) (xy 92.71 148.59)
+		)
+		(stroke
+			(width 0)
+			(type default)
+		)
+	)
 	(wire
 		(pts
@@
 	(wire
 		(pts
+			(xy 95.25 151.13) (xy 97.79 151.13)
+		)
+		(stroke
+			(width 0)
+			(type default)
+		)
+	)
+	(wire
+		(pts
 			(xy 217.17 38.1) (xy 234.95 38.1)
 		)
@@
 	(bus
 		(pts
+			(xy 92.71 144.78) (xy 92.71 146.05)
+		)
+		(stroke
+			(width 0)
+			(type default)
+		)
+	)
+	(bus
+		(pts
 			(xy 49.53 40.64) (xy 49.53 43.18)
 		)
@@
 		)
 	)
+	(bus
+		(pts
+			(xy 92.71 148.59) (xy 92.71 151.13)
+		)
+		(stroke
+			(width 0)
+			(type default)
+		)
+	)
 	(wire
 		(pts
@@
 	(wire
 		(pts
+			(xy 82.55 153.67) (xy 90.17 153.67)
+		)
+		(stroke
+			(width 0)
+			(type default)
+		)
+	)
+	(wire
+		(pts
 			(xy 35.56 48.26) (xy 46.99 48.26)
 		)
@@
 		)
 	)
+	(label "GPIO_[91..96]"
+		(at 92.71 144.78 0)
+		(fields_autoplaced yes)
+		(effects
+			(font
+				(size 1.27 1.27)
+			)
+			(justify left bottom)
+		)
+	)
 	(label "GPIO_29"
 		(at 91.44 30.48 0)
@@
 		)
 	)
+	(label "GPIO_91"
+		(at 97.79 148.59 0)
+		(effects
+			(font
+				(size 1.27 1.27)
+			)
+			(justify left bottom)
+		)
+	)
 	(label "GPIO_33"
 		(at 91.44 40.64 0)
@@
 		)
 	)
+	(label "GPIO_93"
+		(at 97.79 153.67 0)
+		(effects
+			(font
+				(size 1.27 1.27)
+			)
+			(justify left bottom)
+		)
+	)
 	(label "GPIO_25"
 		(at 35.56 106.68 0)
@@
 		)
 	)
+	(label "GPIO_94"
+		(at 82.55 148.59 0)
+		(effects
+			(font
+				(size 1.27 1.27)
+			)
+			(justify left bottom)
+		)
+	)
 	(label "GPIO_39"
 		(at 91.44 66.04 0)
@@
 		)
 	)
+	(label "GPIO_96"
+		(at 82.55 153.67 0)
+		(effects
+			(font
+				(size 1.27 1.27)
+			)
+			(justify left bottom)
+		)
+	)
 	(label "GPIO_65"
 		(at 148.59 63.5 0)
@@
 		)
 	)
+	(label "GPIO_92"
+		(at 97.79 151.13 0)
+		(effects
+			(font
+				(size 1.27 1.27)
+			)
+			(justify left bottom)
+		)
+	)
 	(label "GPIO_[46..54]"
 		(at 105.41 87.63 0)
@@
 		)
 	)
+	(label "GPIO_95"
+		(at 82.55 151.13 0)
+		(effects
+			(font
+				(size 1.27 1.27)
+			)
+			(justify left bottom)
+		)
+	)
 	(label "GPIO_80"
 		(at 148.59 109.22 0)
@@
 			)
 		)
-		(property "Footprint" ""
+		(property "Footprint" "Resistor_SMD:R_0603_1608Metric_Pad0.98x0.95mm_HandSolder"
 			(at 229.87 68.072 90)
 			(effects
@@
 			)
 		)
-		(property "Footprint" ""
+		(property "Footprint" "Resistor_SMD:R_0603_1608Metric_Pad0.98x0.95mm_HandSolder"
 			(at 227.33 121.412 90)
 			(effects
@@
 			)
 		)
-		(property "Footprint" ""
+		(property "Footprint" "Resistor_SMD:R_0603_1608Metric_Pad0.98x0.95mm_HandSolder"
 			(at 222.25 95.758 90)
 			(effects
@@
 			)
 		)
-		(property "Footprint" ""
+		(property "Footprint" "Resistor_SMD:R_0603_1608Metric_Pad0.98x0.95mm_HandSolder"
 			(at 228.6 94.742 90)
 			(effects
@@
 			)
 		)
-		(property "Footprint" ""
+		(property "Footprint" "Resistor_SMD:R_0603_1608Metric_Pad0.98x0.95mm_HandSolder"
 			(at 220.98 122.428 90)
 			(effects
@@
 			)
 		)
-		(property "Footprint" ""
+		(property "Footprint" "Resistor_SMD:R_0603_1608Metric_Pad0.98x0.95mm_HandSolder"
 			(at 223.52 69.088 90)
 			(effects
