File: Puzzle1/puzzle1/puzzle1.kicad_pcb (KiCad board)
At the start: 2 copper layers, 9 parts, among them J1 Conn_01x16_Pin, J2 Conn_01x16_Pin, J3 Raspberry_Pi_2_3, U1 PCA9555D, U2 PCA9555D

Commit message: update
Parts:
- removed R3, R4: 10k, Resistor_SMD:R_0805_2012Metric
- added J10: Conn_01x09_Socket, Connector_JST:JST_XH_B9B-XH-A_1x09_P2.50mm_Vertical, F.Cu at (25.5, 110.8)
- added J11: Conn_01x09_Socket, Connector_JST:JST_XH_B9B-XH-A_1x09_P2.50mm_Vertical, F.Cu at (25.5, 118.6)
- added J4: Conn_01x09_Socket, Connector_JST:JST_XH_B9B-XH-A_1x09_P2.50mm_Vertical, F.Cu at (25.5, 64.0)
- added J5: Conn_01x09_Socket, Connector_JST:JST_XH_B9B-XH-A_1x09_P2.50mm_Vertical, F.Cu at (25.5, 71.8)
- added J6: Conn_01x09_Socket, Connector_JST:JST_XH_B9B-XH-A_1x09_P2.50mm_Vertical, F.Cu at (25.5, 79.6)
- added J7: Conn_01x09_Socket, Connector_JST:JST_XH_B9B-XH-A_1x09_P2.50mm_Vertical, F.Cu at (25.5, 87.4)
- added J8: Conn_01x09_Socket, Connector_JST:JST_XH_B9B-XH-A_1x09_P2.50mm_Vertical, F.Cu at (25.5, 95.2)
- added J9: Conn_01x09_Socket, Connector_JST:JST_XH_B9B-XH-A_1x09_P2.50mm_Vertical, F.Cu at (25.5, 103.0)
- added U3: PCA9555D, Package_SO:SOIC-24W_7.5x15.4mm_P1.27mm, F.Cu at (54.3, 36.5)
- added U4: PCA9555D, Package_SO:SOIC-24W_7.5x15.4mm_P1.27mm, F.Cu at (67.2, 36.5)
- added U5: PCA9555D, Package_SO:SOIC-24W_7.5x15.4mm_P1.27mm, F.Cu at (80.1, 36.5)
- added U6: PCA9555D, Package_SO:SOIC-24W_7.5x15.4mm_P1.27mm, F.Cu at (93.0, 36.5)
- J1: value Conn_01x16_Pin -> Conn_01x04_Pin; footprint Connector_PinSocket_2.54mm:PinSocket_2x09_P2.54mm_Vertical -> Connector_JST:JST_XH_B4B-XH-A_1x04_P2.50mm_Vertical
- J2: value Conn_01x16_Pin -> Conn_01x09_Socket; footprint Connector_PinSocket_2.54mm:PinSocket_2x09_P2.54mm_Vertical -> Connector_JST:JST_XH_B9B-XH-A_1x09_P2.50mm_Vertical
- J3: value Raspberry_Pi_2_3 -> Conn_01x09_Socket; footprint Connector_PinSocket_2.54mm:PinSocket_2x20_P2.54mm_Vertical -> Connector_JST:JST_XH_B9B-XH-A_1x09_P2.50mm_Vertical
- R1, R2: value 10k -> 4.7k; footprint Resistor_SMD:R_0805_2012Metric -> Resistor_SMD:R_0603_1608Metric_Pad0.98x0.95mm_HandSolder
- moved J2 208.8 mm to (25.5, 48.4), turned to 0 degrees
- moved U1 196.3 mm to (28.5, 36.5)
- moved U2 177.9 mm to (41.4, 36.5)
- moved J3 158.2 mm to (25.5, 56.2)
- moved J1 144.8 mm to (105.0, 31.4), turned to 0 degrees
- moved R1 130.4 mm to (103.7, 37.0)
- moved R2 125.8 mm to (103.7, 39.5)
Connections:
- J1 pad 1: Net-(J1-Pin_1) -> +5V
- J1 pad 2: Net-(J1-Pin_2) -> SCL
- J1 pad 3: Net-(J1-Pin_3) -> SDA
- J1 pad 4: Net-(J1-Pin_4) -> GND
- J3 pad 1: +3.3V -> Net-(J3-Pin_1)
- J3 pad 2: +5V -> Net-(J3-Pin_2)
- J3 pad 3: /SDA -> Net-(J3-Pin_3)
- J3 pad 4: +5V -> Net-(J3-Pin_4)
- J3 pad 5: /SCL -> Net-(J3-Pin_5)
- J3 pad 6: GND -> Net-(J3-Pin_6)
- J3 pad 7: unconnected-(J3-GCLK0/GPIO4-Pad7) -> Net-(J3-Pin_7)
- J3 pad 8: unconnected-(J3-GPIO14/TXD-Pad8) -> Net-(J3-Pin_8)
- J3 pad 9: GND -> Net-(J3-Pin_9)
- R1 pad 2: /GPIOExpander1/SCL -> SDA
- R2 pad 2: /GPIOExpander1/SDA -> SCL
- U1 pad 10: Net-(J1-Pin_7) -> Net-(J2-Pin_7)
- U1 pad 11: Net-(J1-Pin_8) -> Net-(J2-Pin_8)
- U1 pad 13: Net-(J1-Pin_9) -> Net-(J2-Pin_9)
- U1 pad 14: Net-(J1-Pin_10) -> Net-(J3-Pin_1)
- U1 pad 15: Net-(J1-Pin_11) -> Net-(J3-Pin_2)
- U1 pad 16: Net-(J1-Pin_12) -> Net-(J3-Pin_3)
- U1 pad 17: Net-(J1-Pin_13) -> Net-(J3-Pin_4)
- U1 pad 18: Net-(J1-Pin_14) -> Net-(J3-Pin_5)
- U1 pad 19: Net-(J1-Pin_15) -> Net-(J3-Pin_6)
- U1 pad 20: Net-(J1-Pin_16) -> Net-(J3-Pin_7)
- U1 pad 21: +5V -> GND
- U1 pad 22: /GPIOExpander1/SCL -> SCL
- U1 pad 23: /GPIOExpander1/SDA -> SDA
- U1 pad 4: Net-(J1-Pin_1) -> Net-(J2-Pin_1)
- U1 pad 5: Net-(J1-Pin_2) -> Net-(J2-Pin_2)
- U1 pad 6: Net-(J1-Pin_3) -> Net-(J2-Pin_3)
- U1 pad 7: Net-(J1-Pin_4) -> Net-(J2-Pin_4)
- U1 pad 8: Net-(J1-Pin_5) -> Net-(J2-Pin_5)
- U1 pad 9: Net-(J1-Pin_6) -> Net-(J2-Pin_6)
- U2 pad 10: Net-(J2-Pin_7) -> Net-(J4-Pin_5)
- U2 pad 11: Net-(J2-Pin_8) -> Net-(J4-Pin_6)
- U2 pad 13: Net-(J2-Pin_9) -> Net-(J4-Pin_7)
- U2 pad 14: Net-(J2-Pin_10) -> Net-(J4-Pin_8)
- U2 pad 15: Net-(J2-Pin_11) -> Net-(J4-Pin_9)
- U2 pad 16: Net-(J2-Pin_12) -> Net-(J5-Pin_1)
- U2 pad 17: Net-(J2-Pin_13) -> Net-(J5-Pin_2)
- U2 pad 18: Net-(J2-Pin_14) -> Net-(J5-Pin_3)
- U2 pad 19: Net-(J2-Pin_15) -> Net-(J5-Pin_4)
- U2 pad 20: Net-(J2-Pin_16) -> Net-(J5-Pin_5)
- U2 pad 22: /GPIOExpander2/SCL -> SCL
- U2 pad 23: /GPIOExpander2/SDA -> SDA
- U2 pad 4: Net-(J2-Pin_1) -> Net-(J3-Pin_8)
- U2 pad 5: Net-(J2-Pin_2) -> Net-(J3-Pin_9)
- U2 pad 6: Net-(J2-Pin_3) -> Net-(J4-Pin_1)
- U2 pad 7: Net-(J2-Pin_4) -> Net-(J4-Pin_2)
- U2 pad 8: Net-(J2-Pin_5) -> Net-(J4-Pin_3)
- U2 pad 9: Net-(J2-Pin_6) -> Net-(J4-Pin_4)
Routing:
- net GND: track 101.3 -> 0.00 mm
- net Net-(J1-Pin_2): track 45.3 -> 0.00 mm
- net Net-(J1-Pin_1): track 44.0 -> 0.00 mm
- net Net-(J2-Pin_2): track 43.8 -> 0.00 mm
- net Net-(J2-Pin_1): track 42.4 -> 0.00 mm
- net Net-(J1-Pin_4): track 41.6 -> 0.00 mm
- net Net-(J2-Pin_4): track 40.6 -> 0.00 mm
- net +5V: track 40.6 -> 0.00 mm, vias 1 -> 0
- net Net-(J1-Pin_3): track 40.3 -> 0.00 mm
- net Net-(J2-Pin_3): track 39.2 -> 0.00 mm
- net Net-(J1-Pin_6): track 38.9 -> 0.00 mm
- net Net-(J1-Pin_5): track 37.2 -> 0.00 mm
- net Net-(J2-Pin_6): track 37.2 -> 0.00 mm
- net Net-(J1-Pin_8): track 36.6 -> 0.00 mm
- net Net-(J2-Pin_5): track 35.4 -> 0.00 mm
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- removed copper zone on F.Cu, net GND

Commit message: update
Parts:
- added J12: Conn_01x04_Socket, Connector_JST:JST_XH_B4B-XH-A_1x04_P2.50mm_Vertical, F.Cu at (160.5, 96.0)
- added J13: Conn_01x04_Socket, Connector_JST:JST_XH_B4B-XH-A_1x04_P2.50mm_Vertical, F.Cu at (160.5, 108.0)
- added J14: Conn_01x04_Socket, Connector_JST:JST_XH_B4B-XH-A_1x04_P2.50mm_Vertical, F.Cu at (160.5, 120.0)
- added R3: 120, Resistor_SMD:R_0603_1608Metric, F.Cu at (142.9, 63.5)
- added R4: 120, Resistor_SMD:R_0603_1608Metric, F.Cu at (145.5, 63.5)
- added R5: 120, Resistor_SMD:R_0603_1608Metric, F.Cu at (148.0, 63.5)
- added R6: 120, Resistor_SMD:R_0603_1608Metric, F.Cu at (150.5, 63.5)
- added R7: 120, Resistor_SMD:R_0603_1608Metric, F.Cu at (155.5, 63.5)
- added R8: 120, Resistor_SMD:R_0603_1608Metric, F.Cu at (153.0, 63.5)
- J11: value Conn_01x09_Socket -> Conn_01x04_Socket; footprint Connector_JST:JST_XH_B9B-XH-A_1x09_P2.50mm_Vertical -> Connector_JST:JST_XH_B4B-XH-A_1x04_P2.50mm_Vertical
- moved J11 125.5 mm to (148.0, 91.5), turned to 90 degrees
- moved J10 122.9 mm to (148.0, 121.0), turned to 90 degrees
- moved J9 94.5 mm to (118.5, 120.0)
- moved J8 93.9 mm to (118.5, 108.0)
- moved J7 93.4 mm to (118.5, 96.0)
- moved J6 93.1 mm to (118.5, 84.0)
- moved J5 80.5 mm to (90.0, 120.0)
- moved J4 78.1 mm to (90.0, 108.0)
- moved J3 75.8 mm to (90.0, 96.0)
- moved J2 73.7 mm to (90.0, 84.0)
- moved U1 65.8 mm to (94.1, 31.4), turned to 90 degrees
- moved U3 62.9 mm to (117.0, 31.5), turned to 90 degrees
- moved U5 59.1 mm to (139.0, 31.5), turned to 90 degrees
- moved U2 54.1 mm to (93.9, 49.4), turned to 90 degrees
- moved U4 51.9 mm to (117.5, 49.5), turned to 90 degrees
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Connections:
- J11 pad 1: Net-(J11-Pin_1) -> +5V
- U6 pad 10: Net-(J11-Pin_6) -> Net-(U6-IO0_6)
- U6 pad 11: Net-(J11-Pin_7) -> Net-(U6-IO0_7)
- U6 pad 13: Net-(J11-Pin_8) -> Net-(U6-IO1_0)
- U6 pad 14: Net-(J11-Pin_9) -> Net-(U6-IO1_1)
- U6 pad 5: Net-(J11-Pin_1) -> Net-(J11-Pin_2)
- U6 pad 6: Net-(J11-Pin_2) -> Net-(J11-Pin_3)
- U6 pad 7: Net-(J11-Pin_3) -> Net-(J11-Pin_4)
- U6 pad 8: Net-(J11-Pin_4) -> Net-(U6-IO0_4)
- U6 pad 9: Net-(J11-Pin_5) -> Net-(U6-IO0_5)
Routing:
- net SCL: track 0.00 -> 164.5 mm, vias 0 -> 2
- net SDA: track 0.00 -> 158.4 mm, vias 0 -> 2
- net Net-(J10-Pin_1): track 0.00 -> 108.5 mm, vias 0 -> 1
- net Net-(J10-Pin_2): track 0.00 -> 104.3 mm, vias 0 -> 1
- net Net-(J10-Pin_3): track 0.00 -> 101.0 mm, vias 0 -> 2
- net Net-(J10-Pin_4): track 0.00 -> 100.8 mm, vias 0 -> 1
- net Net-(J10-Pin_8): track 0.00 -> 95.5 mm, vias 0 -> 2
- net Net-(J10-Pin_7): track 0.00 -> 86.3 mm, vias 0 -> 1
- net Net-(J14-Pin_2): track 0.00 -> 59.8 mm, vias 0 -> 1
- net Net-(J14-Pin_1): track 0.00 -> 57.7 mm, vias 0 -> 2
- net Net-(J10-Pin_9): track 0.00 -> 51.7 mm
- net Net-(J13-Pin_1): track 0.00 -> 49.8 mm, vias 0 -> 1
- net Net-(J13-Pin_2): track 0.00 -> 49.8 mm, vias 0 -> 1
- net Net-(J11-Pin_2): track 0.00 -> 39.1 mm
- net Net-(J12-Pin_1): track 0.00 -> 38.9 mm
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- added copper zone on F.Cu, net +5V
- added copper zone on B.Cu, net GND
Other:
- board outline added: 120 x 115 mm

Commit message: update
working on PCB layout
Parts:
- moved J11 198.7 mm to (-35.0, 14.2), turned to 0 degrees
- moved J9 187.6 mm to (-62.0, 68.8)
- moved J8 186.5 mm to (-62.0, 61.0)
- moved J7 185.5 mm to (-62.0, 53.2)
- moved J6 184.6 mm to (-62.0, 45.4)
- moved J5 172.9 mm to (-62.0, 37.6)
- moved J4 170.9 mm to (-62.0, 29.8)
- moved J3 169.1 mm to (-62.0, 22.0)
- moved J2 167.3 mm to (-62.0, 14.2)
- moved J14 133.5 mm to (35.5, 73.0)
- moved R7 120.0 mm to (35.5, 63.7)
- moved R8 115.0 mm to (38.0, 63.7)
- moved J13 110.7 mm to (55.5, 73.0)
- moved R5 92.5 mm to (55.5, 63.5)
- moved R6 92.5 mm to (58.0, 63.5)
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Routing:
- net SDA: track 158.4 -> 41.2 mm, vias 2 -> 0
- net SCL: track 164.5 -> 51.4 mm, vias 2 -> 0
- net Net-(J10-Pin_1): track 108.5 -> 2.56 mm, vias 1 -> 0
- net Net-(J10-Pin_2): track 104.3 -> 4.07 mm, vias 1 -> 0
- net Net-(J10-Pin_3): track 101.0 -> 5.75 mm, vias 2 -> 0
- net Net-(J10-Pin_4): track 100.8 -> 7.43 mm, vias 1 -> 0
- net Net-(J10-Pin_8): track 95.5 -> 12.0 mm, vias 2 -> 0
- net Net-(J10-Pin_7): track 86.3 -> 10.3 mm, vias 1 -> 0
- net Net-(J14-Pin_2): track 59.8 -> 8.50 mm, vias 1 -> 0
- net Net-(J14-Pin_1): track 57.7 -> 8.50 mm, vias 2 -> 0
- net Net-(J13-Pin_1): track 49.8 -> 8.68 mm, vias 1 -> 0
- net Net-(J13-Pin_2): track 49.8 -> 8.67 mm, vias 1 -> 0
- net Net-(J10-Pin_9): track 51.7 -> 13.8 mm
- net GND: track 34.2 -> 0.00 mm, vias 1 -> 17
- net Net-(J12-Pin_1): track 38.9 -> 8.68 mm
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- removed copper zone on F.Cu, net +5V
- removed copper zone on B.Cu, net GND
Other:
- board outline removed

Commit message: update
Parts:
- moved J1 82.1 mm to (37.5, 29.0), turned to 90 degrees
- moved R1 73.3 mm to (49.1, 22.6), turned to -90 degrees
- moved R2 69.1 mm to (49.0, 27.6), turned to 90 degrees

Commit message: pre-check
Parts:
- moved J7 192.4 mm to (127.0, 89.0), turned to -90 degrees
- moved J9 189.3 mm to (127.0, 59.0), turned to -90 degrees
- moved J8 181.5 mm to (113.0, 109.0), turned to 90 degrees
- moved J11 166.9 mm to (129.5, 42.0)
- moved J4 119.1 mm to (49.0, 73.0), turned to -90 degrees
- moved J2 114.7 mm to (49.0, 43.0), turned to -90 degrees
- moved J5 111.7 mm to (35.0, 93.0), turned to 90 degrees
- moved J6 110.2 mm to (32.0, 103.0)
- moved J3 105.3 mm to (35.0, 63.0), turned to 90 degrees
- moved U6 101.5 mm to (90.3, 55.0)
- moved U5 89.8 mm to (90.0, 75.0)
- moved U4 87.0 mm to (90.0, 95.0)
- moved J13 85.6 mm to (129.5, 30.0)
- moved U3 85.2 mm to (71.0, 95.0)
- moved J14 83.9 mm to (113.5, 42.0)
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Routing:
- net SDA: track 41.2 -> 133.8 mm, vias 0 -> 3
- net SCL: track 51.4 -> 124.8 mm
- net +5V: track 0.00 -> 63.9 mm, vias 0 -> 17
- net Net-(J7-Pin_1): track 8.65 -> 59.0 mm
- net Net-(J7-Pin_8): track 8.70 -> 57.9 mm
- net Net-(J9-Pin_8): track 5.34 -> 52.7 mm
- net Net-(J11-Pin_4): track 10.4 -> 57.2 mm
- net Net-(J5-Pin_3): track 8.77 -> 54.1 mm, vias 0 -> 1
- net 9: track 10.1 -> 55.3 mm
- net Net-(J7-Pin_3): track 12.0 -> 56.8 mm
- net Net-(J11-Pin_3): track 10.5 -> 54.2 mm
- net Net-(J7-Pin_2): track 10.3 -> 53.4 mm, vias 0 -> 1
- net Net-(J5-Pin_2): track 11.1 -> 52.3 mm
- net Net-(J3-Pin_1): track 4.74 -> 45.8 mm, vias 0 -> 1
- net Net-(J9-Pin_9): track 3.65 -> 44.6 mm
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- added copper zone on F.Cu, net +5V
- added copper zone on B.Cu, net GND
Other:
- board outline added: 125 x 100 mm

Commit message: update after review
Parts:
- added C1: 100n, Capacitor_SMD:C_0603_1608Metric_Pad1.08x0.95mm_HandSolder, F.Cu at (49.1, 56.5)
- added C2: 100n, Capacitor_SMD:C_0603_1608Metric_Pad1.08x0.95mm_HandSolder, F.Cu at (69.1, 56.5)
- added C3: 100n, Capacitor_SMD:C_0603_1608Metric_Pad1.08x0.95mm_HandSolder, F.Cu at (89.1, 56.5)
- added C4: 100n, Capacitor_SMD:C_0603_1608Metric_Pad1.08x0.95mm_HandSolder, F.Cu at (109.1, 56.5)
- added C5: 100n, Capacitor_SMD:C_0603_1608Metric_Pad1.08x0.95mm_HandSolder, F.Cu at (129.1, 56.5)
- added C6: 100n, Capacitor_SMD:C_0603_1608Metric_Pad1.08x0.95mm_HandSolder, F.Cu at (149.1, 56.5)
- J10, J2, J3, J4, J5, J6, J7, J8, J9: value Conn_01x09_Socket -> Conn_01x09_Pin
- J11, J12, J13, J14: value Conn_01x04_Socket -> Conn_01x04_Pin
- R3, R4, R5, R6, R7, R8: footprint Resistor_SMD:R_0603_1608Metric -> Resistor_SMD:R_0603_1608Metric_Pad0.98x0.95mm_HandSolder
- moved J5 95.5 mm to (130.5, 93.0), turned to 0 degrees
- moved R3 93.5 mm to (90.0, 123.1), turned to -90 degrees
- moved R4 90.5 mm to (95.0, 123.1), turned to 90 degrees
- moved J11 89.2 mm to (75.5, 113.0)
- moved R5 87.6 mm to (105.0, 123.1), turned to -90 degrees
- moved J13 86.4 mm to (105.5, 113.0)
- moved J12 86.1 mm to (90.5, 113.0)
- moved R6 85.4 mm to (110.0, 123.1), turned to 90 degrees
- moved R8 85.1 mm to (125.0, 123.1), turned to 90 degrees
- moved R1 84.1 mm to (29.5, 105.6), turned to 90 degrees
- moved R7 80.9 mm to (120.0, 123.1), turned to -90 degrees
- moved J1 79.7 mm to (37.5, 99.5), turned to -90 degrees
- moved R2 77.9 mm to (29.5, 100.9), turned to -90 degrees
- moved J10 73.4 mm to (48.0, 113.0), turned to 0 degrees
- moved J14 71.3 mm to (120.5, 113.0)
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Connections:
- net +5V renamed VCC
- net 1 renamed /Connectors/GPIO_64
- net 6 renamed /Connectors/GPIO_33
- net 7 renamed /Connectors/GPIO_34
- net 8 renamed /Connectors/GPIO_35
- net 9 renamed /Connectors/GPIO_36
- net Net-(J10-Pin_1) renamed /Connectors/GPIO_73
- net Net-(J10-Pin_2) renamed /Connectors/GPIO_74
- net Net-(J10-Pin_3) renamed /Connectors/GPIO_75
- net Net-(J10-Pin_4) renamed /Connectors/GPIO_76
- net Net-(J10-Pin_5) renamed /Connectors/GPIO_77
- net Net-(J10-Pin_6) renamed /Connectors/GPIO_78
- net Net-(J10-Pin_7) renamed /Connectors/GPIO_79
- net Net-(J10-Pin_8) renamed /Connectors/GPIO_80
- net Net-(J10-Pin_9) renamed /Connectors/GPIO_81
- net Net-(J11-Pin_2) renamed /Connectors/GPIO_82
- net Net-(J11-Pin_3) renamed /Connectors/GPIO_83
- net Net-(J11-Pin_4) renamed /Connectors/GPIO_84
- net Net-(J2-Pin_1) renamed /Connectors/GPIO_1
- net Net-(J2-Pin_2) renamed /Connectors/GPIO_2
- net Net-(J2-Pin_3) renamed /Connectors/GPIO_3
- net Net-(J2-Pin_4) renamed /Connectors/GPIO_4
- net Net-(J2-Pin_5) renamed /Connectors/GPIO_5
- net Net-(J2-Pin_6) renamed /Connectors/GPIO_6
- net Net-(J2-Pin_7) renamed /Connectors/GPIO_7
- net Net-(J2-Pin_8) renamed /Connectors/GPIO_8
- net Net-(J2-Pin_9) renamed /Connectors/GPIO_9
- net Net-(J3-Pin_1) renamed /Connectors/GPIO_10
- net Net-(J3-Pin_2) renamed /Connectors/GPIO_11
- net Net-(J3-Pin_3) renamed /Connectors/GPIO_12
- net Net-(J3-Pin_4) renamed /Connectors/GPIO_13
- net Net-(J3-Pin_5) renamed /Connectors/GPIO_14
- net Net-(J3-Pin_6) renamed /Connectors/GPIO_15
- net Net-(J3-Pin_7) renamed /Connectors/GPIO_16
- net Net-(J3-Pin_8) renamed /Connectors/GPIO_17
- net Net-(J3-Pin_9) renamed /Connectors/GPIO_18
- net Net-(J4-Pin_1) renamed /Connectors/GPIO_19
- net Net-(J4-Pin_2) renamed /Connectors/GPIO_20
- net Net-(J4-Pin_3) renamed /Connectors/GPIO_21
- net Net-(J4-Pin_4) renamed /Connectors/GPIO_22
- net Net-(J4-Pin_5) renamed /Connectors/GPIO_23
- net Net-(J4-Pin_6) renamed /Connectors/GPIO_24
- net Net-(J4-Pin_7) renamed /Connectors/GPIO_25
- net Net-(J4-Pin_8) renamed /Connectors/GPIO_26
- net Net-(J4-Pin_9) renamed /Connectors/GPIO_27
- net Net-(J5-Pin_1) renamed /Connectors/GPIO_28
- net Net-(J5-Pin_2) renamed /Connectors/GPIO_29
- net Net-(J5-Pin_3) renamed /Connectors/GPIO_30
- net Net-(J5-Pin_4) renamed /Connectors/GPIO_31
- net Net-(J5-Pin_5) renamed /Connectors/GPIO_32
- net Net-(J6-Pin_1) renamed /Connectors/GPIO_37
- net Net-(J6-Pin_2) renamed /Connectors/GPIO_38
- net Net-(J6-Pin_3) renamed /Connectors/GPIO_39
- net Net-(J6-Pin_4) renamed /Connectors/GPIO_40
- net Net-(J6-Pin_5) renamed /Connectors/GPIO_41
- net Net-(J6-Pin_6) renamed /Connectors/GPIO_42
- net Net-(J6-Pin_7) renamed /Connectors/GPIO_43
- net Net-(J6-Pin_8) renamed /Connectors/GPIO_44
- net Net-(J6-Pin_9) renamed /Connectors/GPIO_45
- net Net-(J7-Pin_1) renamed /Connectors/GPIO_46
- net Net-(J7-Pin_2) renamed /Connectors/GPIO_47
- net Net-(J7-Pin_3) renamed /Connectors/GPIO_48
- net Net-(J7-Pin_4) renamed /Connectors/GPIO_49
- net Net-(J7-Pin_5) renamed /Connectors/GPIO_50
- net Net-(J7-Pin_6) renamed /Connectors/GPIO_51
- net Net-(J7-Pin_7) renamed /Connectors/GPIO_52
- net Net-(J7-Pin_8) renamed /Connectors/GPIO_53
- net Net-(J7-Pin_9) renamed /Connectors/GPIO_54
- net Net-(J8-Pin_1) renamed /Connectors/GPIO_55
- net Net-(J8-Pin_2) renamed /Connectors/GPIO_56
- net Net-(J8-Pin_3) renamed /Connectors/GPIO_57
- net Net-(J8-Pin_4) renamed /Connectors/GPIO_58
- net Net-(J8-Pin_5) renamed /Connectors/GPIO_59
- net Net-(J8-Pin_6) renamed /Connectors/GPIO_60
- net Net-(J8-Pin_7) renamed /Connectors/GPIO_61
- net Net-(J8-Pin_8) renamed /Connectors/GPIO_62
- net Net-(J8-Pin_9) renamed /Connectors/GPIO_63
- net Net-(J9-Pin_2) renamed /Connectors/GPIO_65
- net Net-(J9-Pin_3) renamed /Connectors/GPIO_66
- net Net-(J9-Pin_4) renamed /Connectors/GPIO_67
- net Net-(J9-Pin_5) renamed /Connectors/GPIO_68
- net Net-(J9-Pin_6) renamed /Connectors/GPIO_69
- net Net-(J9-Pin_7) renamed /Connectors/GPIO_70
- net Net-(J9-Pin_8) renamed /Connectors/GPIO_71
- net Net-(J9-Pin_9) renamed /Connectors/GPIO_72
- net Net-(U6-IO0_4) renamed /Connectors/GPIO_85
- net Net-(U6-IO0_6) renamed /Connectors/GPIO_87
- net Net-(U6-IO1_0) renamed /Connectors/GPIO_89
- net SCL renamed /SCL
- net SDA renamed /SDA
- R4 pad 1: Net-(J12-Pin_2) -> /Connectors/GPIO_86
- R4 pad 2: Net-(U6-IO0_5) -> Net-(J12-Pin_2)
- R6 pad 1: Net-(J13-Pin_2) -> /Connectors/GPIO_88
- R6 pad 2: Net-(U6-IO0_7) -> Net-(J13-Pin_2)
- R8 pad 1: Net-(J14-Pin_2) -> /Connectors/GPIO_90
- R8 pad 2: Net-(U6-IO1_1) -> Net-(J14-Pin_2)
- U6 pad 11: Net-(U6-IO0_7) -> /Connectors/GPIO_88
- U6 pad 14: Net-(U6-IO1_1) -> /Connectors/GPIO_90
- U6 pad 15: unconnected-(U6-IO1_2-Pad15) -> /Connectors/GPIO_91
- U6 pad 16: unconnected-(U6-IO1_3-Pad16) -> /Connectors/GPIO_92
- U6 pad 17: unconnected-(U6-IO1_4-Pad17) -> /Connectors/GPIO_93
- U6 pad 18: unconnected-(U6-IO1_5-Pad18) -> /Connectors/GPIO_94
- U6 pad 19: unconnected-(U6-IO1_6-Pad19) -> /Connectors/GPIO_95
- U6 pad 20: unconnected-(U6-IO1_7-Pad20) -> /Connectors/GPIO_96
- U6 pad 9: Net-(U6-IO0_5) -> /Connectors/GPIO_86
Routing:
- net /Connectors/GPIO_86: track 0.00 -> 119.8 mm, vias 0 -> 2
- net /Connectors/GPIO_88: track 0.00 -> 103.1 mm, vias 0 -> 2
- net /Connectors/GPIO_85: track 35.4 -> 126.4 mm
- net /Connectors/GPIO_74: track 20.8 -> 110.8 mm, vias 0 -> 1
- net /Connectors/GPIO_73: track 19.6 -> 109.4 mm, vias 0 -> 1
- net /Connectors/GPIO_75: track 21.3 -> 110.6 mm
- net /Connectors/GPIO_76: track 21.8 -> 109.9 mm
- net /Connectors/GPIO_77: track 21.7 -> 109.1 mm
- net /Connectors/GPIO_78: track 22.3 -> 109.7 mm
- net /Connectors/GPIO_80: track 23.2 -> 106.3 mm
- net /Connectors/GPIO_79: track 23.3 -> 105.9 mm
- net /Connectors/GPIO_87: track 31.1 -> 109.1 mm
- net /Connectors/GPIO_90: track 0.00 -> 77.2 mm, vias 0 -> 2
- net /Connectors/GPIO_81: track 36.1 -> 112.3 mm, vias 0 -> 1
- net GND: track 27.3 -> 96.7 mm, vias 15 -> 16
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Other:
- board size 125 x 100 mm -> 135 x 85 mm
- copper layers 2 -> 4

Commit message: added base board to designs, not fully done yet
weekend update
Parts:
- added G***: LOGO, Library:PhantomVaultPCBLogo5cmBackside, F.Cu at (98.8, 79.8)
- added H1: MountingHole_Pad, MountingHole:MountingHole_3.2mm_M3_DIN965_Pad, F.Cu at (155.0, 121.5)
- added H2: MountingHole_Pad, MountingHole:MountingHole_3.2mm_M3_DIN965_Pad, F.Cu at (30.0, 121.5)
- added H3: MountingHole_Pad, MountingHole:MountingHole_3.2mm_M3_DIN965_Pad, F.Cu at (30.0, 58.0)
- renumbered J1 to Input, J12 to LED1, J13 to LED2, J14 to LED3, J2 to Row1, J3 to Row2, J4 to Row3, J5 to Row4, J6 to Row5, J7 to Row6, J8 to Row7, J9 to Row8, J10 to Row9, J11 to WireTriggers
Other:
- board size 135 x 85 mm -> 135 x 73.6 mm
- board text added: "1"
- board text added: "2"
- board text added: "3"
- board text added: "4"
- board text added: "GND"
- board text added: "Gre"
- board text added: "Red"
- board text added: "SCL"
- board text added: "SDA"
- board text added: "VCC"
- board text added: "Wire1"
- board text added: "Wire2"
- board text added: "Wire3"
- board text added: "www.phantomvault.nl Puzzle1 interface PCB Version: 1.0 Engineer: CCO"
