File: BaseBoard/BaseBoard/BaseBoard.kicad_sch (KiCad schematic)
At the start: 18 parts, among them J1 Screw_Terminal_01x02, J2 Conn_01x06_Pin, Q1 2N3904, Q2 2N3904, U1 WT32-ETH01, U2 LMR51430

Commit message: zitten fout in
zitten fout in, niet gebruiken
Parts:
- added J3: Conn_01x04_Pin, Connector_JST:JST_XH_B4B-XH-A_1x04_P2.50mm_Vertical, symbol Connector:Conn_01x04_Pin
- added J4: Conn_01x10_Pin, Connector_PinHeader_2.54mm:PinHeader_1x10_P2.54mm_Vertical, symbol Connector:Conn_01x10_Pin
- added J5: Screw_Terminal_01x02, TerminalBlock_Phoenix:TerminalBlock_Phoenix_MKDS-3-2-5.08_1x02_P5.08mm_Horizontal, symbol Connector:Screw_Terminal_01x02
- L1: footprint generic:L0603 -> Inductor_SMD:L_Bourns_SDR0604; Field5 (none) -> SDE0604A-6R8M
- U1: footprint WT32-ETH01:WT32-ETH01 -> PhantomVault:WT32-ETH01-M
Connections:
- net +5V: now also J3.1 (Pin_1), J5.1 (Pin_1)
- net GND: now also U1.14 (GND), U1.23 (GND), J3.4 (Pin_4), J5.2 (Pin_2)
- net +3.3V: now reaches U1.3 (3.3V)
- net +3.3V: no longer U1.10 (3.3V)
- net at U1.15 (IO2/ADC2_CH2/TCH2/PRG_FLOAT_OR_GND): now also J4.3 (Pin_3)
- net at U1.16 (IO4/ADC2_CH0/TCH0): now also J4.4 (Pin_4)
- net at U1.17 (IO35/ADC1_CH7/INPUT_ONLY): now also J4.5 (Pin_5)
- net at U1.18 (IO12/ADC2_CH5/TCH5/BOOT_FLOAT_OR_LOW): now also J4.6 (Pin_6)
- net at U1.19 (IO14/ADC2_CH6/TCH6): now also J4.7 (Pin_7)
- net at U1.20 (IO15/ADC2_CH3/TCH3): now also J4.8 (Pin_8)
- net at U1.21 (IO36/ADC1_CH0/INPUT_ONLY): now also J4.9 (Pin_9)
- net at U1.22 (IO39/ADC1_CH3/INPUT_ONLY): now also J4.10 (Pin_10)
- net at U1.4 (ESP32_EN): now also J4.2 (Pin_2)
- net at U1.5 (IO32/ADC1_CH4/TCH9): now also J3.3 (Pin_3)
- net at U1.6 (IO33/ADC1_CH5/TCH8): now also J3.2 (Pin_2)
- net at U1.7 (IO5/BOOT_FLOAT): now also J4.1 (Pin_1)
- new net +3V3: U1.10 (3.3V)
- no-connect marks 0 -> 2
Other:
- moved on the sheet: H1, H2, H3
